Commit message: pkg name updated

File: urdf/materials.xacro (robot description, xacro)
@@ -1,4 +1,4 @@
 <?xml version="1.0" ?>
-<robot name="ty_sensor_mount" xmlns:xacro="http://www.ros.org/wiki/xacro" >
+<robot name="ty_sensors_mount" xmlns:xacro="http://www.ros.org/wiki/xacro" >
 <material name="ty_color">
   <color rgba="0.700 0.700 0.700 1.000"/>

File: urdf/tracker.urdf.xacro (robot description, xacro)
@@ -20,5 +20,5 @@
         <origin xyz="0.0 0 0.1" rpy="1.57 0 1.57"/>
         <geometry>
-          <mesh filename="package://ty_sensor_mount/meshes/realsense_t265.stl" scale="0.001 0.001 0.001"  />
+          <mesh filename="package://ty_sensors_mount/meshes/realsense_t265.stl" scale="0.001 0.001 0.001"  />
         </geometry>
         <material name="Grey">

File: urdf/ty_sensors_mount.urdf (robot description, URDF)
Before this commit: robot ty_sensor_mount, 12 links, 11 joints
Links:
- link lidar: geometry collision mesh filename=package://ty_sensors_mount/meshes/lidar.stl scale=0.001 0.001 0.001; visual mesh filename=package://ty_sensors_mount/meshes/lidar.stl scale=0.001 0.001 0.001
- link lidar_base: geometry collision mesh filename=package://ty_sensors_mount/meshes/lidar_base.stl scale=0.001 0.001 0.001; visual mesh filename=package://ty_sensors_mount/meshes/lidar_base.stl scale=0.001 0.001 0.001
- link realsense_link: geometry visual mesh filename=package://ty_sensors_mount/meshes/realsense_t265.stl scale=0.001 0.001 0.001
- link sensor_mount_base: geometry collision mesh filename=package://ty_sensors_mount/meshes/sensor_mount_base.stl scale=0.001 0.001 0.001; visual mesh filename=package://ty_sensors_mount/meshes/sensor_mount_base.stl scale=0.001 0.001 0.001

File: urdf/ty_sensors_mount.xacro (robot description, xacro)
@@ -1,10 +1,10 @@
 <?xml version="1.0"?>
-<robot name="ty_sensor_mount" xmlns:xacro="http://www.ros.org/wiki/xacro">
+<robot name="ty_sensors_mount" xmlns:xacro="http://www.ros.org/wiki/xacro">
   <xacro:property name="deg_to_rad" value="0.01745329251994329577" />
-  <xacro:include filename="$(find ty_sensor_mount)/urdf/materials.xacro" />
-  <xacro:include filename="$(find ty_sensor_mount)/gazebo/ty_sensor_mount_materials.gazebo" />
-  <xacro:include filename="$(find ty_sensor_mount)/gazebo/ty_sensor_mount_physics.gazebo" />
-  <xacro:include filename="$(find ty_sensor_mount)/gazebo/ty_sensor_mount_plugins.gazebo" />
-  <xacro:include filename="$(find ty_sensor_mount)/urdf/tracker.urdf.xacro" />
+  <xacro:include filename="$(find ty_sensors_mount)/urdf/materials.xacro" />
+  <xacro:include filename="$(find ty_sensors_mount)/gazebo/ty_sensors_mount_materials.gazebo" />
+  <xacro:include filename="$(find ty_sensors_mount)/gazebo/ty_sensors_mount_physics.gazebo" />
+  <xacro:include filename="$(find ty_sensors_mount)/gazebo/ty_sensors_mount_plugins.gazebo" />
+  <xacro:include filename="$(find ty_sensors_mount)/urdf/tracker.urdf.xacro" />
   <xacro:macro name="ty_sensor" params="name:=ty_sensor parent *origin">
     <link name="sensor_mount_base">
@@ -17,5 +17,5 @@
         <origin rpy="0 0 0" xyz="0 0 0" />
         <geometry>
-          <mesh filename="package://ty_sensor_mount/meshes/sensor_mount_base.stl" scale="0.001 0.001 0.001" />
+          <mesh filename="package://ty_sensors_mount/meshes/sensor_mount_base.stl" scale="0.001 0.001 0.001" />
         </geometry>
         <material name="ty_color" />
@@ -24,5 +24,5 @@
         <origin rpy="0 0 0" xyz="0 0 0" />
         <geometry>
-          <mesh filename="package://ty_sensor_mount/meshes/sensor_mount_base.stl" scale="0.001 0.001 0.001" />
+          <mesh filename="package://ty_sensors_mount/meshes/sensor_mount_base.stl" scale="0.001 0.001 0.001" />
         </geometry>
       </collision>
@@ -37,5 +37,5 @@
         <origin rpy="0 0 0" xyz="0.062 0.02 -0.1524" />
         <geometry>
-          <mesh filename="package://ty_sensor_mount/meshes/lidar_base.stl" scale="0.001 0.001 0.001" />
+          <mesh filename="package://ty_sensors_mount/meshes/lidar_base.stl" scale="0.001 0.001 0.001" />
         </geometry>
         <material name="ty_color" />
@@ -44,5 +44,5 @@
         <origin rpy="0 0 0" xyz="0.062 0.02 -0.1524" />
         <geometry>
-          <mesh filename="package://ty_sensor_mount/meshes/lidar_base.stl" scale="0.001 0.001 0.001" />
+          <mesh filename="package://ty_sensors_mount/meshes/lidar_base.stl" scale="0.001 0.001 0.001" />
         </geometry>
       </collision>
@@ -57,5 +57,5 @@
         <origin rpy="0 0 0" xyz="0.02 -0.0 -0.2001" />
         <geometry>
-          <mesh filename="package://ty_sensor_mount/meshes/lidar.stl" scale="0.001 0.001 0.001" />
+          <mesh filename="package://ty_sensors_mount/meshes/lidar.stl" scale="0.001 0.001 0.001" />
         </geometry>
         <material name="ty_color" />
@@ -64,5 +64,5 @@
         <origin rpy="0 0 0" xyz="0.02 -0.0 -0.2001" />
         <geometry>
-          <mesh filename="package://ty_sensor_mount/meshes/lidar.stl" scale="0.001 0.001 0.001" />
+          <mesh filename="package://ty_sensors_mount/meshes/lidar.stl" scale="0.001 0.001 0.001" />
         </geometry>
       </collision>
